Commit message: feat: side comments erased

File: pepper_description/urdf/pepper1.0_generated_urdf/pepperGazebo.xacro (robot description, xacro)
@@ -3,87 +3,4 @@
     <!-- MACROS FOR DISABLE LINKS -->
 	<xacro:property name="PI" value="3.14159265359" />
-    <!-- <xacro:macro name="DisabledLinks" params="side side_small">
-        <plugin name="${side}Finger11_link" filename="libroboticsgroup_gazebo_disable_link_plugin.so">
-            <link>${side}Finger11_link</link>
-        </plugin>
-        <plugin name="${side}Finger12_link" filename="libroboticsgroup_gazebo_disable_link_plugin.so">
-            <link>${side}Finger12_link</link>
-        </plugin>
-        <plugin name="${side}Finger13_link" filename="libroboticsgroup_gazebo_disable_link_plugin.so">
-            <link>${side}Finger13_link</link>
-        </plugin>
-        <plugin name="${side}Finger21_link" filename="libroboticsgroup_gazebo_disable_link_plugin.so">
-            <link>${side}Finger21_link</link>
-        </plugin>
-        <plugin name="${side}Finger22_link" filename="libroboticsgroup_gazebo_disable_link_plugin.so">
-            <link>${side}Finger22_link</link>
-        </plugin>
-        <plugin name="${side}Finger23_link" filename="libroboticsgroup_gazebo_disable_link_plugin.so">
-            <link>${side}Finger23_link</link>
-        </plugin>
-        <plugin name="${side}Finger31_link" filename="libroboticsgroup_gazebo_disable_link_plugin.so">
-            <link>${side}Finger31_link</link>
-        </plugin>
-        <plugin name="${side}Finger32_link" filename="libroboticsgroup_gazebo_disable_link_plugin.so">
-            <link>${side}Finger32_link</link>
-        </plugin>
-        <plugin name="${side}Finger33_link" filename="libroboticsgroup_gazebo_disable_link_plugin.so">
-            <link>${side}Finger33_link</link>
-        </plugin>
-        <plugin name="${side}Finger41_link" filename="libroboticsgroup_gazebo_disable_link_plugin.so">
-            <link>${side}Finger41_link</link>
-        </plugin>
-        <plugin name="${side}Finger42_link" filename="libroboticsgroup_gazebo_disable_link_plugin.so">
-            <link>${side}Finger42_link</link>
-        </plugin>
-        <plugin name="${side}Finger43_link" filename="libroboticsgroup_gazebo_disable_link_plugin.so">
-            <link>${side}Finger43_link</link>
-        </plugin>
-        <plugin name="${side}Thumb1_link" filename="libroboticsgroup_gazebo_disable_link_plugin.so">
-            <link>${side}Thumb1_link</link>
-        </plugin>
-        <plugin name="${side}Thumb2_link" filename="libroboticsgroup_gazebo_disable_link_plugin.so">
-            <link>${side}Thumb2_link</link>
-        </plugin>
-        <plugin name="${side_small}_gripper" filename="libroboticsgroup_gazebo_disable_link_plugin.so">
-            <link>${side_small}_gripper</link>
-        </plugin>
-    </xacro:macro>  -->
-    <!-- MACROS FOR MIMIC JOINTS -->
-    <!-- Fingers -->
- <!--    <xacro:macro name="FingerMimics" params="side num">
-        <plugin name="mimic_${side}Finger${num}1" filename="libroboticsgroup_gazebo_mimic_joint_plugin.so">
-            <joint>${side}Hand</joint>
-            <mimicJoint>${side}Finger${num}1</mimicJoint>
-            <multiplier>-${PI/4}</multiplier>
-            <offset>${PI/4}</offset>
-        </plugin>
-        <plugin name="mimic_${side}Finger${num}2" filename="libroboticsgroup_gazebo_mimic_joint_plugin.so">
-            <joint>${side}Hand</joint>
-            <mimicJoint>${side}Finger${num}2</mimicJoint>
-            <multiplier>-${PI/4}</multiplier>
-            <offset>${PI/4}</offset>
-        </plugin>
-        <plugin name="mimic_${side}Finger${num}3" filename="libroboticsgroup_gazebo_mimic_joint_plugin.so">
-            <joint>${side}Hand</joint>
-            <mimicJoint>${side}Finger${num}3</mimicJoint>
-            <multiplier>-${PI/4}</multiplier>
-            <offset>${PI/4}</offset>
-        </plugin>
-    </xacro:macro>
-    <xacro:macro name="ThumbMimics" params="side">
-        <plugin name="${side}Thumb1" filename="libroboticsgroup_gazebo_mimic_joint_plugin.so">
-            <joint>${side}Hand</joint>
-            <mimicJoint>${side}Thumb1</mimicJoint>
-            <multiplier>-${PI/4}</multiplier>
-            <offset>${PI/4}</offset>
-        </plugin>
-        <plugin name="${side}Thumb2" filename="libroboticsgroup_gazebo_mimic_joint_plugin.so">
-            <joint>${side}Hand</joint>
-            <mimicJoint>${side}Thumb2</mimicJoint>
-            <multiplier>-${PI/4}</multiplier>
-            <offset>${PI/4}</offset>
-        </plugin>
-    </xacro:macro> -->
     <!-- GAZEBO ROS CONTROL -->
     <gazebo>
@@ -93,16 +10,4 @@
             <robotSimType>gazebo_ros_control/DefaultRobotHWSim</robotSimType>
         </plugin>
- <!--        <xacro:FingerMimics side="L" num="1"/>
-        <xacro:FingerMimics side="L" num="2"/>
-        <xacro:FingerMimics side="L" num="3"/>
-        <xacro:FingerMimics side="L" num="4"/>
-        <xacro:FingerMimics side="R" num="1"/>
-        <xacro:FingerMimics side="R" num="2"/>
-        <xacro:FingerMimics side="R" num="3"/>
-        <xacro:FingerMimics side="R" num="4"/>
-        <xacro:ThumbMimics side="L"/>
-        <xacro:ThumbMimics side="R"/>
-        <xacro:DisabledLinks side="L" side_small="l"/>
-        <xacro:DisabledLinks side="R" side_small="r"/>  -->
     </gazebo>
     <!-- END OF GAZEBO ROS CONTROL PLUGIN -->

File: pepper_description/urdf/pepper1.0_generated_urdf/pepperGazeboCPU_no_arms.xacro (robot description, xacro)
@@ -3,87 +3,4 @@
     <!-- MACROS FOR DISABLE LINKS -->
 	<xacro:property name="PI" value="3.14159265359" />
-    <!-- <xacro:macro name="DisabledLinks" params="side side_small">
-        <plugin name="${side}Finger11_link" filename="libroboticsgroup_gazebo_disable_link_plugin.so">
-            <link>${side}Finger11_link</link>
-        </plugin>
-        <plugin name="${side}Finger12_link" filename="libroboticsgroup_gazebo_disable_link_plugin.so">
-            <link>${side}Finger12_link</link>
-        </plugin>
-        <plugin name="${side}Finger13_link" filename="libroboticsgroup_gazebo_disable_link_plugin.so">
-            <link>${side}Finger13_link</link>
-        </plugin>
-        <plugin name="${side}Finger21_link" filename="libroboticsgroup_gazebo_disable_link_plugin.so">
-            <link>${side}Finger21_link</link>
-        </plugin>
-        <plugin name="${side}Finger22_link" filename="libroboticsgroup_gazebo_disable_link_plugin.so">
-            <link>${side}Finger22_link</link>
-        </plugin>
-        <plugin name="${side}Finger23_link" filename="libroboticsgroup_gazebo_disable_link_plugin.so">
-            <link>${side}Finger23_link</link>
-        </plugin>
-        <plugin name="${side}Finger31_link" filename="libroboticsgroup_gazebo_disable_link_plugin.so">
-            <link>${side}Finger31_link</link>
-        </plugin>
-        <plugin name="${side}Finger32_link" filename="libroboticsgroup_gazebo_disable_link_plugin.so">
-            <link>${side}Finger32_link</link>
-        </plugin>
-        <plugin name="${side}Finger33_link" filename="libroboticsgroup_gazebo_disable_link_plugin.so">
-            <link>${side}Finger33_link</link>
-        </plugin>
-        <plugin name="${side}Finger41_link" filename="libroboticsgroup_gazebo_disable_link_plugin.so">
-            <link>${side}Finger41_link</link>
-        </plugin>
-        <plugin name="${side}Finger42_link" filename="libroboticsgroup_gazebo_disable_link_plugin.so">
-            <link>${side}Finger42_link</link>
-        </plugin>
-        <plugin name="${side}Finger43_link" filename="libroboticsgroup_gazebo_disable_link_plugin.so">
-            <link>${side}Finger43_link</link>
-        </plugin>
-        <plugin name="${side}Thumb1_link" filename="libroboticsgroup_gazebo_disable_link_plugin.so">
-            <link>${side}Thumb1_link</link>
-        </plugin>
-        <plugin name="${side}Thumb2_link" filename="libroboticsgroup_gazebo_disable_link_plugin.so">
-            <link>${side}Thumb2_link</link>
-        </plugin>
-        <plugin name="${side_small}_gripper" filename="libroboticsgroup_gazebo_disable_link_plugin.so">
-            <link>${side_small}_gripper</link>
-        </plugin>
-    </xacro:macro>  -->
-    <!-- MACROS FOR MIMIC JOINTS -->
-    <!-- Fingers -->
- <!--    <xacro:macro name="FingerMimics" params="side num">
-        <plugin name="mimic_${side}Finger${num}1" filename="libroboticsgroup_gazebo_mimic_joint_plugin.so">
-            <joint>${side}Hand</joint>
-            <mimicJoint>${side}Finger${num}1</mimicJoint>
-            <multiplier>-${PI/4}</multiplier>
-            <offset>${PI/4}</offset>
-        </plugin>
-        <plugin name="mimic_${side}Finger${num}2" filename="libroboticsgroup_gazebo_mimic_joint_plugin.so">
-            <joint>${side}Hand</joint>
-            <mimicJoint>${side}Finger${num}2</mimicJoint>
-            <multiplier>-${PI/4}</multiplier>
-            <offset>${PI/4}</offset>
-        </plugin>
-        <plugin name="mimic_${side}Finger${num}3" filename="libroboticsgroup_gazebo_mimic_joint_plugin.so">
-            <joint>${side}Hand</joint>
-            <mimicJoint>${side}Finger${num}3</mimicJoint>
-            <multiplier>-${PI/4}</multiplier>
-            <offset>${PI/4}</offset>
-        </plugin>
-    </xacro:macro>
-    <xacro:macro name="ThumbMimics" params="side">
-        <plugin name="${side}Thumb1" filename="libroboticsgroup_gazebo_mimic_joint_plugin.so">
-            <joint>${side}Hand</joint>
-            <mimicJoint>${side}Thumb1</mimicJoint>
-            <multiplier>-${PI/4}</multiplier>
-            <offset>${PI/4}</offset>
-        </plugin>
-        <plugin name="${side}Thumb2" filename="libroboticsgroup_gazebo_mimic_joint_plugin.so">
-            <joint>${side}Hand</joint>
-            <mimicJoint>${side}Thumb2</mimicJoint>
-            <multiplier>-${PI/4}</multiplier>
-            <offset>${PI/4}</offset>
-        </plugin>
-    </xacro:macro> -->
     <!-- GAZEBO ROS CONTROL -->
     <gazebo>
@@ -93,16 +10,4 @@
             <robotSimType>gazebo_ros_control/DefaultRobotHWSim</robotSimType>
         </plugin>
- <!--        <xacro:FingerMimics side="L" num="1"/>
-        <xacro:FingerMimics side="L" num="2"/>
-        <xacro:FingerMimics side="L" num="3"/>
-        <xacro:FingerMimics side="L" num="4"/>
-        <xacro:FingerMimics side="R" num="1"/>
-        <xacro:FingerMimics side="R" num="2"/>
-        <xacro:FingerMimics side="R" num="3"/>
-        <xacro:FingerMimics side="R" num="4"/>
-        <xacro:ThumbMimics side="L"/>
-        <xacro:ThumbMimics side="R"/>
-        <xacro:DisabledLinks side="L" side_small="l"/>
-        <xacro:DisabledLinks side="R" side_small="r"/>  -->
     </gazebo>
     <!-- END OF GAZEBO ROS CONTROL PLUGIN -->

File: pepper_description/urdf/pepper1.0_generated_urdf/pepperTransmission_no_arms.xacro (robot description, xacro)
@@ -76,17 +76,5 @@
 			</actuator>
 		</transmission>
-        <!-- Disabling hands as they cant do much in simulation anyways -->
-<!-- 		<transmission name="${side}Hand_Transmission">
-			<type>transmission_interface/SimpleTransmission</type>
-			<joint name="${side}Hand">
-  			  <hardwareInterface>hardware_interface/VelocityJointInterface</hardwareInterface>
-            </joint>
-			<actuator name="${side}Hand_Motor">
-				<mechanicalReduction>${speed_red_type3B}</mechanicalReduction>
-			</actuator>
-		</transmission> -->
 		</xacro:macro>
-	<!-- <xacro:arm_joints_transmissions side="L"/>
-	<xacro:arm_joints_transmissions side="R"/> -->
 	<!-- LEGS -->
 	<transmission name="HipRoll_Transmission">
@@ -117,19 +105,3 @@
                 </actuator>
         </transmission>
-        <!-- XACRO -->
-        <!-- Disabling wheels, given they are not used in simulation anymore -->
-<!--         <xacro:macro name="wheel_joints_transmissions" params="side">
-                <transmission name="Wheel${side}_Transmission">
-                        <type>transmission_interface/SimpleTransmission</type>
-                        <joint name="Wheel${side}">
-                                <hardwareInterface>EffortJointInterface</hardwareInterface>
-                        </joint>
-                        <actuator name="Wheel${side}_Motor">
-                                <mechanicalReduction>${speed_red_type5B}</mechanicalReduction>
-                        </actuator>
-                </transmission>
-        </xacro:macro>
-        <xacro:wheel_joints_transmissions side="FL"/>
-        <xacro:wheel_joints_transmissions side="B"/>
-        <xacro:wheel_joints_transmissions side="FR"/> -->
 </robot>
